File: KiCad/VoltageCurrentMeter.sch (KiCad schematic (older format))
At the start: 22 parts, among them J1 CHAN-1, J10 Power Jumper, J11 Daughter Board 1, J12 Daughter Board 2, J2 CHAN-2, J3 CHAN-3, J4 CHAN-4, J5 CHAN-5, J6 CHAN-6, J7 CHAN-7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

Commit message: Updates to schematic and added images and a README.
Parts:
- J9: value V In -> V-IN GND
Changed lines of the file:
@@
 P 4850 5250
 F 0 "J9" H 4850 4900 50  0000 C CNN
-F 1 "V In" H 4850 5000 50  0000 C CNN
+F 1 "V-IN    GND" H 5150 5200 50  0000 C CNN
 F 2 "TerminalBlock_Phoenix:TerminalBlock_Phoenix_MKDS-1,5-2-5.08_1x02_P5.08mm_Horizontal" H 4850 5250 50  0001 C CNN
 F 3 "~" H 4850 5250 50  0001 C CNN
@@
 U 1 1 61A860F2
 P 5600 5150
-F 0 "J10" H 5600 5150 50  0000 R CNN
+F 0 "J10" H 5800 4650 50  0000 R CNN
 F 1 "Power Jumper" H 5950 4750 50  0000 R CNN
 F 2 "Connector_PinHeader_2.54mm:PinHeader_1x03_P2.54mm_Vertical" H 5600 5150 50  0001 C CNN
